Commit message: feat: added oltf_data_aq.py for aquaring transfer function

File: armstrong_ws/src/armstrong_description/urdf/armstrong_v1/base.urdf.xacro (robot description, xacro)
@@ -5,12 +5,12 @@
     <xacro:property name="base_dy" value="0.2" />
     <xacro:property name="base_dz" value="0.3" />
-    <xacro:property name="link1_mass" value="0.5" />
-    <xacro:property name="link1_length" value="0.5" />
+    <xacro:property name="link1_mass" value="200" />
+    <xacro:property name="link1_length" value="1.2" />
     <xacro:property name="link1_radius" value="0.05" />
-    <xacro:property name="link2_mass" value="0.3" />
-    <xacro:property name="link2_length" value="0.4" />
+    <xacro:property name="link2_mass" value="280" />
+    <xacro:property name="link2_length" value="1.6" />
     <xacro:property name="link2_radius" value="0.04" />
     <xacro:property name="tooltip_radius" value="0.1" />
-    <xacro:property name="tooltip_mass" value="0.01" />
+    <xacro:property name="tooltip_mass" value="20" />
     <xacro:macro name="cylinder_inertia" params="mass radius length">
         <inertia ixx="${mass * (3*radius*radius + length*length) / 12.0}"

Commit message: feat: add effort_teleop feature

File: armstrong_ws/src/armstrong_description/urdf/armstrong_v1/base.urdf.xacro (robot description, xacro)
@@ -1,16 +1,16 @@
 <?xml version="1.0"?>
 <robot xmlns:xacro="http://www.ros.org/wiki/xacro">
-    <xacro:property name="base_mass" value="100.0" />
-    <xacro:property name="base_dx" value="0.2" />
-    <xacro:property name="base_dy" value="0.2" />
+    <xacro:property name="base_mass" value="10000.0" />
+    <xacro:property name="base_dx" value="0.5" />
+    <xacro:property name="base_dy" value="0.5" />
     <xacro:property name="base_dz" value="0.3" />
-    <xacro:property name="link1_mass" value="200" />
-    <xacro:property name="link1_length" value="1.2" />
-    <xacro:property name="link1_radius" value="0.05" />
-    <xacro:property name="link2_mass" value="280" />
-    <xacro:property name="link2_length" value="1.6" />
-    <xacro:property name="link2_radius" value="0.04" />
-    <xacro:property name="tooltip_radius" value="0.1" />
-    <xacro:property name="tooltip_mass" value="20" />
+    <xacro:property name="link1_mass" value="40" />
+    <xacro:property name="link1_length" value="1.6" />
+    <xacro:property name="link1_radius" value="0.15" />
+    <xacro:property name="link2_mass" value="25" />
+    <xacro:property name="link2_length" value="1.2" />
+    <xacro:property name="link2_radius" value="0.1" />
+    <xacro:property name="tooltip_radius" value="0.25" />
+    <xacro:property name="tooltip_mass" value="1" />
     <xacro:macro name="cylinder_inertia" params="mass radius length">
         <inertia ixx="${mass * (3*radius*radius + length*length) / 12.0}"
@@ -54,5 +54,5 @@
         <origin xyz="0 0 ${base_dz/2}" rpy="0 0 0" />
         <axis xyz="0 1 0" />
-        <limit lower="${-pi/2}" upper="${pi/2}" effort="100" velocity="3.0" />
+        <limit lower="${-pi/3}" upper="${pi/3}" effort="1000" velocity="3.0" />
         <dynamics damping="0.1" friction="0.1"/>
     </joint>
@@ -81,5 +81,5 @@
         <origin xyz="0 0 ${link1_length}" rpy="0 0 0" />
         <axis xyz="0 1 0" />
-        <limit lower="${-pi/2}" upper="${pi/2}" effort="50" velocity="3.0" />
+        <limit lower="${-pi/2}" upper="${pi/2}" effort="200" velocity="3.0" />
         <dynamics damping="0.1" friction="0.1"/>
     </joint>

File: armstrong_ws/src/armstrong_description/urdf/armstrong_v1/ros2_control.urdf.xacro (robot description, xacro)
@@ -16,6 +16,6 @@
         <joint name="joint2">
             <command_interface name="effort">
-                <param name="min">-50</param>
-                <param name="max">50</param>
+                <param name="min">-200</param>
+                <param name="max">200</param>
             </command_interface>
             <state_interface name="position"/>

Commit message: feat: modified oltf test and teleop, and removed build (forgot to ignore)

File: armstrong_ws/src/armstrong_description/urdf/armstrong_v1/base.urdf.xacro (robot description, xacro)
@@ -5,4 +5,8 @@
     <xacro:property name="base_dy" value="0.5" />
     <xacro:property name="base_dz" value="0.3" />
+    <!-- <xacro:property name="joint1_type" value="fixed" /> -->
+    <xacro:property name="joint1_type" value="revolute" />
+    <!-- <xacro:property name="joint2_type" value="fixed" /> -->
+    <xacro:property name="joint2_type" value="revolute" />
     <xacro:property name="link1_mass" value="40" />
     <xacro:property name="link1_length" value="1.6" />
@@ -49,10 +53,10 @@
         </inertial>
     </link>
-    <joint name="joint1" type="revolute">
+    <joint name="joint1" type="${joint1_type}">
         <parent link="base_link" />
         <child link="link1" />
         <origin xyz="0 0 ${base_dz/2}" rpy="0 0 0" />
         <axis xyz="0 1 0" />
-        <limit lower="${-pi/3}" upper="${pi/3}" effort="1000" velocity="3.0" />
+        <limit lower="${-pi/2 + pi/4}" upper="${pi/2 - pi/4}" effort="1000" velocity="3.0" />
         <dynamics damping="0.1" friction="0.1"/>
     </joint>
@@ -76,5 +80,5 @@
         </inertial>
     </link>
-    <joint name="joint2" type="revolute">
+    <joint name="joint2" type="${joint2_type}">
         <parent link="link1" />
         <child link="link2" />

Commit message: feat: added and modified system identification codes

File: armstrong_ws/src/armstrong_description/urdf/armstrong_v1/base.urdf.xacro (robot description, xacro)
@@ -1,11 +1,10 @@
 <?xml version="1.0"?>
 <robot xmlns:xacro="http://www.ros.org/wiki/xacro">
+    <xacro:arg name="lock_joint1_arg" default="true" />
     <xacro:property name="base_mass" value="10000.0" />
     <xacro:property name="base_dx" value="0.5" />
     <xacro:property name="base_dy" value="0.5" />
     <xacro:property name="base_dz" value="0.3" />
-    <!-- <xacro:property name="joint1_type" value="fixed" /> -->
     <xacro:property name="joint1_type" value="revolute" />
-    <!-- <xacro:property name="joint2_type" value="fixed" /> -->
     <xacro:property name="joint2_type" value="revolute" />
     <xacro:property name="link1_mass" value="40" />
@@ -58,5 +57,12 @@
         <origin xyz="0 0 ${base_dz/2}" rpy="0 0 0" />
         <axis xyz="0 1 0" />
-        <limit lower="${-pi/2 + pi/4}" upper="${pi/2 - pi/4}" effort="1000" velocity="3.0" />
+        <!-- Conditional limits for joint1 -->
+        <xacro:if value="${$(arg lock_joint1_arg)}">
+            <limit lower="0" upper="0" effort="1000" velocity="3.0" />
+        </xacro:if>
+        <xacro:unless value="${$(arg lock_joint1_arg)}">
+            <limit lower="${-pi/2 + pi/4}" upper="${pi/2 - pi/4}" effort="1000" velocity="3.0" />
+        </xacro:unless>
+        <limit lower="0" upper="0" effort="1000" velocity="3.0" />
         <dynamics damping="0.1" friction="0.1"/>
     </joint>
@@ -85,5 +91,5 @@
         <origin xyz="0 0 ${link1_length}" rpy="0 0 0" />
         <axis xyz="0 1 0" />
-        <limit lower="${-pi/2}" upper="${pi/2}" effort="200" velocity="3.0" />
+        <limit lower="${-pi/2}" upper="${pi/2}" effort="300" velocity="3.0" />
         <dynamics damping="0.1" friction="0.1"/>
     </joint>
